File: PhaserPedalBoard/Digital.kicad_sch (KiCad schematic)
At the start: 19 parts, among them J1 Footswitch, J2 SWD Header, SW2 RST, U6 STM32L052K6Tx, U7 LM2904

Commit message: rough schematic
Parts:
- added C25, C26: 1n, symbol Device:C
- added D10, D11, D8, D9: Orange, LED_THT:LED_D3.0mm, symbol Device:LED
- added Q1: BC847, Package_TO_SOT_SMD:SOT-23, symbol Transistor_BJT:BC847
- added Q2, Q3, Q7: 2N7002, Package_TO_SOT_SMD:SOT-23, symbol Transistor_FET:2N7002
- added R47: 1k, symbol Device:R_US
- added R48, R49, R50: 470, Resistor_SMD:R_0805_2012Metric, symbol Device:R_US
- added R51, R52: 10k, symbol Device:R_US
- added RV1, RV2: 10kB, Potentiometer_THT:Potentiometer_Alpha_RD901F-40-00D_Single_Vertical_CircularHoles, symbol Device:R_Potentiometer_US
- R43: value 1Meg -> 82k
- R44: value 1Meg -> 91k
- U6: value STM32L052K6Tx -> STM32L052K6T6
Connections:
- net +3.3V: now also R48.1, R49.1, R50.1
- net +3.3VA: now also RV1.3, RV2.3
- net BypLED: now also Q2.1 (G)
- net GND: now also C25.2, C26.2, Q2.2 (S), Q3.2 (S), Q7.2 (S), R47.1, RV1.1, RV2.1
- net KnobLED: now also Q3.1 (G)
- net ShapeADC: now also C26.1, R52.2
- net SpeedADC: now also C25.1, R51.2
- net TapLED: now also Q7.1 (G)
- net at R43.2, U7.2 (-): now also R44.1; no longer R44.2
- net DAC_OUT: now reaches U7.1
- net DAC_OUT: now also R44.2, U7.5 (+)
- net at U7.6 (-): now also Q1.2 (E), R47.2
- net at U7.7: now also Q1.1 (B)
- new net: D8.2 (A), R48.2
- new net: D9.1 (K), Q1.3 (C)
- new net: D11.2 (A), R50.2
- new net: R52.1, RV2.2
- new net: D10.2 (A), R49.2
- new net: R51.1, RV1.2
- new net: D10.1 (K), Q3.3 (D)
- new net: D8.1 (K), Q2.3 (D)
- new net: D11.1 (K), Q7.3 (D)
- new net +12V: D9.2 (A)
- no-connect marks 0 -> 15
Other:
- note added: "DAC output stage"
- note added: "LEDs"
- note added: "MCU- STM32L052K6T6"
- moved on the sheet: C19, C20, C21, C22, C23, C4, J1, J2, R35, R36, R37, R4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

Commit message: schematic hygiene
Parts:
- added C27: 1u, symbol Device:C
- added J8: (no value), Connector:BatteryContact_Keystone_243, symbol Connector:GroundingSpring
- added R53: 8k2, symbol Device:R_US
- added TP10: VDAC, TestPoint:TestPoint_THTPad_D2.0mm_Drill1.0mm_VAL, symbol Connector:TestPoint
- added TP11: SPD, TestPoint:TestPoint_THTPad_D2.0mm_Drill1.0mm_VAL, symbol Connector:TestPoint
- added TP12: SHP, TestPoint:TestPoint_THTPad_D2.0mm_Drill1.0mm_VAL, symbol Connector:TestPoint
- added TP5: DAC, TestPoint:TestPoint_THTPad_D2.0mm_Drill1.0mm_VAL, symbol Connector:TestPoint
- R44: value 91k -> 100k
Connections:
- net DAC_OUT: now also TP5.1
- net GND: now also C27.2, J8.1
- net ShapeADC: now also TP12.1
- net SpeedADC: now also TP11.1
- net Vdac: now also R53.1, TP10.1; no longer R43.1
- new net: C27.1, R43.1, R53.2
Other:
- note added: "Control pots"
- note added: "Footswitch header"
- note added: "Test points"
- moved on the sheet: C19, C20, C21, C22, C23, C25, C26, C4, J1, J2, R35, R36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

Commit message: rough layout
Parts:
- removed D10, D11: Orange, LED_THT:LED_D3.0mm, symbol Device:LED
- removed Q3, Q7: 2N7002, Package_TO_SOT_SMD:SOT-23, symbol Transistor_FET:2N7002
- removed R49, R50: 470, Resistor_SMD:R_0805_2012Metric, symbol Device:R_US
- removed TP10: VDAC, TestPoint:TestPoint_THTPad_D2.0mm_Drill1.0mm_VAL, symbol Connector:TestPoint
- removed TP11: SPD, TestPoint:TestPoint_THTPad_D2.0mm_Drill1.0mm_VAL, symbol Connector:TestPoint
- removed TP12: SHP, TestPoint:TestPoint_THTPad_D2.0mm_Drill1.0mm_VAL, symbol Connector:TestPoint
- added J5: In, Connector_Audio:Jack_6.35mm_Tayda_PJ664C_Mono_Horizontal, symbol Connector_Audio:AudioJack2_Switch
- added J6: Out, Connector_Audio:Jack_6.35mm_Tayda_PJ664C_Mono_Horizontal, symbol Connector_Audio:AudioJack2_Switch
- C19, C20, C21, C22, C23, C25, C26, C27, C4: footprint (none) -> Capacitor_SMD:C_0805_2012Metric
- J1: footprint (none) -> Connector_PinHeader_2.54mm:PinHeader_1x06_P2.54mm_Vertical
- R4, R43, R44, R45, R46, R47, R51, R52, R53: footprint (none) -> Resistor_SMD:R_0805_2012Metric
- RV1, RV2: footprint Potentiometer_THT:Potentiometer_Alpha_RD901F-40-00D_Single_Vertical_CircularHoles -> Potentiometer_THT:Potentiometer_Alpha_RV16AF_42_Single_Long
Connections:
- net +12V is gone; now on an unnamed net: D9.2 (A)
- net +12VA: now also D8.2 (A)
- net BypLED: now also U6.25 (PA15); no longer U6.26 (PB3)
- net FX_IN: now also J5.T
- net FX_OUT: now also J6.T
- net GND: now also J5.S, J5.SN, J6.S, J6.SN
- net ShapeADC: now also U6.7 (PA1); no longer U6.8 (PA2)
- net SpeedADC: now also U6.8 (PA2); no longer U6.7 (PA1)
- net at R48.2: no longer D8.2 (A)
- net at D9.1 (K): now also Q2.3 (D); no longer Q1.3 (C)
- net at D8.1 (K): now also Q1.3 (C); no longer Q2.3 (D)
- net KnobLED: no longer names the net of U6.28 (PB5)
- net TapLED: no longer names the net of U6.27 (PB4)
- no-connect marks 15 -> 19
Other:
- moved on the sheet: C19, C20, C21, C22, C4, D8, D9, J1, J2, R35, R36, R37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

Commit message: routed, DRC passing
Parts:
- removed TP5: DAC, TestPoint:TestPoint_THTPad_D2.0mm_Drill1.0mm_VAL, symbol Connector:TestPoint
Changed lines of the file:
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@@
 	(wire
 		(pts
-			(xy 201.93 127) (xy 201.93 129.54)
-		)
-		(stroke
-			(width 0)
-			(type default)
-		)
-	)
-	(wire
-		(pts
 			(xy 27.813 54.61) (xy 31.623 54.61)
 		)
@@
 		)
 	)
-	(global_label "DAC_OUT"
-		(shape input)
-		(at 201.93 129.54 0)
-		(fields_autoplaced yes)
-		(effects
-			(font
-				(size 1.27 1.27)
-			)
-			(justify left)
-		)
-		(property "Intersheetrefs" "${INTERSHEET_REFS}"
-			(at 213.14 129.54 0)
-			(hide yes)
-			(show_name no)
-			(do_not_autoplace no)
-			(effects
-				(font
-					(size 1.27 1.27)
-				)
-				(justify left)
-			)
-		)
-	)
 	(global_label "FX_OUT"
 		(shape input)
@@
 					(unit 1)
 				)
-			)
-		)
-	)
-	(symbol
-		(lib_id "Connector:TestPoint")
-		(at 201.93 127 0)
-		(unit 1)
-		(body_style 1)
-		(exclude_from_sim no)
-		(in_bom no)
-		(on_board yes)
-		(in_pos_files yes)
-		(dnp no)
-		(fields_autoplaced yes)
-		(property "Reference" "TP5"
-			(at 204.216 122.4279 0)
-			(show_name no)
-			(do_not_autoplace no)
-			(effects
-				(font
-					(size 1.27 1.27)
-				)
-				(justify left)
-			)
-		)
-		(property "Value" "DAC"
-			(at 204.216 124.9679 0)
-			(show_name no)
-			(do_not_autoplace no)
-			(effects
-				(font
-					(size 1.27 1.27)
-				)
-				(justify left)
-			)
-		)
-		(property "Footprint" "TestPoint:TestPoint_THTPad_D2.0mm_Drill1.0mm_VAL"
-			(at 207.01 127 0)
-			(hide yes)
-			(show_name no)
-			(do_not_autoplace no)
-			(effects
-				(font
-					(size 1.27 1.27)
-				)
-			)
-		)
-		(property "Datasheet" ""
-			(at 207.01 127 0)
-			(hide yes)
-			(show_name no)
-			(do_not_autoplace no)
-			(effects
-				(font
-					(size 1.27 1.27)
-				)
-			)
-		)
-		(property "Description" "test point"
-			(at 201.93 127 0)
-			(hide yes)
-			(show_name no)
-			(do_not_autoplace no)
-			(effects
-				(font
-					(size 1.27 1.27)
-				)
-			)
-		)
-		(pin "1"
-		)
-		(instances
-			(project "PhaserPedalBoard"
-				(path "/121c4899-4e95-4dc0-b332-63e8ed3089d8/337bd860-9d0a-468c-ab48-5592dad52d55"
-					(reference "TP5")
-					(unit 1)
-				)

Commit message: routing w DRC passing
Parts:
- removed C21: 10u, Capacitor_SMD:C_0805_2012Metric, symbol Device:C
Connections:
- net BypLED: now also U6.14 (PB0); no longer U6.25 (PA15)
Changed lines of the file:
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@@
 	)
 	(junction
-		(at 84.963 31.75)
-		(diameter 0)
-		(color 0 0 0 0)
-	)
-	(junction
 		(at 65.913 31.75)
 		(diameter 0)
@@
 	)
 	(no_connect
+		(at 93.98 87.63)
+	)
+	(no_connect
 		(at 63.5 80.01)
 	)
@@
 		(at 76.962 119.126)
 	)
-	(no_connect
-		(at 63.5 67.31)
-	)
-	(wire
-		(pts
-			(xy 84.963 39.37) (xy 84.963 40.64)
-		)
-		(stroke
-			(width 0)
-			(type default)
-		)
-	)
 	(wire
 		(pts
@@
 	(wire
 		(pts
+			(xy 59.436 67.31) (xy 63.5 67.31)
+		)
+		(stroke
+			(width 0)
+			(type default)
+		)
+	)
+	(wire
+		(pts
 			(xy 27.813 46.99) (xy 30.353 46.99)
 		)
@@
 	(wire
 		(pts
-			(xy 104.902 87.63) (xy 93.98 87.63)
-		)
-		(stroke
-			(width 0)
-			(type default)
-		)
-	)
-	(wire
-		(pts
 			(xy 27.813 49.53) (xy 27.813 48.26)
 		)
@@
 	(wire
 		(pts
-			(xy 84.963 31.75) (xy 95.123 31.75)
+			(xy 81.153 31.75) (xy 95.123 31.75)
 		)
 		(stroke
@@
 	(wire
 		(pts
-			(xy 81.153 31.75) (xy 84.963 31.75)
-		)
-		(stroke
-			(width 0)
-			(type default)
-		)
-	)
-	(wire
-		(pts
 			(xy 45.593 54.61) (xy 46.863 54.61)
 		)
@@
 	)
 	(label "BypLED"
-		(at 104.902 87.63 0)
+		(at 59.436 67.31 180)
 		(effects
 			(font
 				(size 1.27 1.27)
 			)
-			(justify left bottom)
+			(justify right bottom)
 		)
 	)
@@
 	)
 	(symbol
-		(lib_id "Device:C")
-		(at 84.963 35.56 0)
-		(unit 1)
-		(body_style 1)
-		(exclude_from_sim no)
-		(in_bom yes)
-		(on_board yes)
-		(in_pos_files yes)
-		(dnp no)
-		(fields_autoplaced yes)
-		(property "Reference" "C21"
-			(at 88.265 34.2899 0)
-			(show_name no)
-			(do_not_autoplace no)
-			(effects
-				(font
-					(size 1.27 1.27)
-				)
-				(justify left)
-			)
-		)
-		(property "Value" "10u"
-			(at 88.265 36.8299 0)
-			(show_name no)
-			(do_not_autoplace no)
-			(effects
-				(font
-					(size 1.27 1.27)
-				)
-				(justify left)
-			)
-		)
-		(property "Footprint" "Capacitor_SMD:C_0805_2012Metric"
-			(at 85.9282 39.37 0)
-			(hide yes)
-			(show_name no)
-			(do_not_autoplace no)
-			(effects
-				(font
-					(size 1.27 1.27)
-				)
-			)
-		)
-		(property "Datasheet" ""
-			(at 84.963 35.56 0)
-			(hide yes)
-			(show_name no)
-			(do_not_autoplace no)
-			(effects
-				(font
-					(size 1.27 1.27)
-				)
-			)
-		)
-		(property "Description" "Unpolarized capacitor"
-			(at 84.963 35.56 0)
-			(hide yes)
-			(show_name no)
-			(do_not_autoplace no)
-			(effects
-				(font
-					(size 1.27 1.27)
-				)
-			)
-		)
-		(pin "2"
-		)
-		(pin "1"
-		)
-		(instances
-			(project "PhaserPedalBoard"
-				(path "/121c4899-4e95-4dc0-b332-63e8ed3089d8/337bd860-9d0a-468c-ab48-5592dad52d55"
-					(reference "C21")
-					(unit 1)
-				)
-			)
-		)
-	)
-	(symbol
 		(lib_id "power:+3.3V")
 		(at 27.94 128.524 0)
@@
 					(unit 1)
 				)
-			)
-		)
-	)
-	(symbol
-		(lib_id "power:GND")
-		(at 84.963 40.64 0)
-		(unit 1)
-		(body_style 1)
-		(exclude_from_sim no)
-		(in_bom yes)
-		(on_board yes)
-		(in_pos_files yes)
-		(dnp no)
-		(fields_autoplaced yes)
-		(property "Reference" "#PWR039"
-			(at 84.963 46.99 0)
-			(hide yes)
-			(show_name no)
-			(do_not_autoplace no)
-			(effects
-				(font
-					(size 1.27 1.27)
-				)
-			)
-		)
-		(property "Value" "GND"
-			(at 84.963 44.45 0)
-			(hide yes)
-			(show_name no)
-			(do_not_autoplace no)
-			(effects
-				(font
-					(size 1.27 1.27)
-				)
-			)
-		)
-		(property "Footprint" ""
-			(at 84.963 40.64 0)
-			(hide yes)
-			(show_name no)
-			(do_not_autoplace no)
-			(effects
-				(font
-					(size 1.27 1.27)
-				)
-			)
-		)
-		(property "Datasheet" ""
-			(at 84.963 40.64 0)
-			(hide yes)
-			(show_name no)
-			(do_not_autoplace no)
-			(effects
-				(font
-					(size 1.27 1.27)
-				)
-			)
-		)
-		(property "Description" "Power symbol creates a global label with name \"GND\" , ground"
-			(at 84.963 40.64 0)
-			(hide yes)
-			(show_name no)
-			(do_not_autoplace no)
-			(effects
-				(font
-					(size 1.27 1.27)
-				)
-			)
-		)
-		(pin "1"
-		)
-		(instances
-			(project "PhaserPedalBoard"
-				(path "/121c4899-4e95-4dc0-b332-63e8ed3089d8/337bd860-9d0a-468c-ab48-5592dad52d55"
-					(reference "#PWR039")
-					(unit 1)
-				)
