File: PhaserPedalBoard/Power.kicad_sch (KiCad schematic)
At the start: 19 parts, among them J2 IO, U1 LMR62014XMF, U4 AMS1117

Commit message: cap values tweak
Parts:
- removed C125: 100u, Capacitor_THT:CP_Radial_D5.0mm_P2.00mm, symbol Device:C_Polarized_US
- added C25: 10u, Capacitor_SMD:C_0805_2012Metric, symbol Device:C
Connections:
- net -9V: now also C25.1
- net GND: now also C25.2
Changed lines of the file:
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@@
-	)
-	(symbol
-		(lib_id "Device:C_Polarized_US")
-		(at 31.75 40.132 0)
-		(unit 1)
-		(body_style 1)
-		(exclude_from_sim no)
-		(in_bom yes)
-		(on_board yes)
-		(in_pos_files yes)
-		(dnp no)
-		(property "Reference" "C125"
-			(at 27.94 38.2269 0)
-			(show_name no)
-			(do_not_autoplace no)
-			(effects
-				(font
-					(size 1.27 1.27)
-				)
-				(justify right)
-			)
-		)
-		(property "Value" "100u"
-			(at 27.94 40.7669 0)
-			(show_name no)
-			(do_not_autoplace no)
-			(effects
-				(font
-					(size 1.27 1.27)
-				)
-				(justify right)
-			)
-		)
-		(property "Footprint" "Capacitor_THT:CP_Radial_D5.0mm_P2.00mm"
-			(at 31.75 40.132 0)
-			(hide yes)
-			(show_name no)
-			(do_not_autoplace no)
-			(effects
-				(font
-					(size 1.27 1.27)
-				)
-			)
-		)
-		(property "Datasheet" ""
-			(at 31.75 40.132 0)
-			(hide yes)
-			(show_name no)
-			(do_not_autoplace no)
-			(effects
-				(font
-					(size 1.27 1.27)
-				)
-			)
-		)
-		(property "Description" "Polarized capacitor, US symbol"
-			(at 31.75 40.132 0)
-			(hide yes)
-			(show_name no)
-			(do_not_autoplace no)
-			(effects
-				(font
-					(size 1.27 1.27)
-				)
-			)
-		)
-		(pin "2"
-		)
-		(pin "1"
-		)
-		(instances
-			(project "PhaserPedalBoard"
-				(path "/121c4899-4e95-4dc0-b332-63e8ed3089d8/90bb61a7-a0ad-417b-bedc-65bd7068296f"
-					(reference "C125")
-					(unit 1)
-				)
-			)
-		)
 	)
 	(symbol
@@
 					(unit 1)
 				)
+			)
+		)
+	)
+	(symbol
+		(lib_id "Device:C")
+		(at 31.75 40.132 0)
+		(mirror x)
+		(unit 1)
+		(body_style 1)
+		(exclude_from_sim no)
+		(in_bom yes)
+		(on_board yes)
+		(in_pos_files yes)
+		(dnp no)
+		(property "Reference" "C25"
+			(at 27.94 38.862 0)
+			(show_name no)
+			(do_not_autoplace no)
+			(effects
+				(font
+					(size 1.27 1.27)
+				)
+				(justify right)
+			)
+		)
+		(property "Value" "10u"
+			(at 27.94 41.402 0)
+			(show_name no)
+			(do_not_autoplace no)
+			(effects
+				(font
+					(size 1.27 1.27)
+				)
+				(justify right)
+			)
+		)
+		(property "Footprint" "Capacitor_SMD:C_0805_2012Metric"
+			(at 32.7152 36.322 0)
+			(hide yes)
+			(show_name no)
+			(do_not_autoplace no)
+			(effects
+				(font
+					(size 1.27 1.27)
+				)
+			)
+		)
+		(property "Datasheet" ""
+			(at 31.75 40.132 0)
+			(hide yes)
+			(show_name no)
+			(do_not_autoplace no)
+			(effects
+				(font
+					(size 1.27 1.27)
+				)
+			)
+		)
+		(property "Description" ""
+			(at 31.75 40.132 0)
+			(hide yes)
+			(show_name no)
+			(do_not_autoplace no)
+			(effects
+				(font
+					(size 1.27 1.27)
+				)
+			)
+		)
+		(property "MPN" "KGM21AR50J106KU"
+			(at 31.75 40.132 0)
+			(hide yes)
+			(show_name no)
+			(do_not_autoplace no)
+			(effects
+				(font
+					(size 1.27 1.27)
+				)
+			)
+		)
+		(property "Purchase Link" "https://www.mouser.com/en/ProductDetail/KYOCERA-AVX/KGM21AR50J106KU?qs=sGAEpiMZZMsh%252B1woXyUXj17cMikWvs6%2FrABKtrcTr%252BA%3D"
+			(at 31.75 40.132 0)
+			(hide yes)
+			(show_name no)
+			(do_not_autoplace no)
+			(effects
+				(font
+					(size 1.27 1.27)
+				)
+			)
+		)
+		(property "KLC_S3.3" ""
+			(at 31.75 40.132 0)
+			(hide yes)
+			(show_name no)
+			(do_not_autoplace no)
+			(effects
+				(font
+					(size 1.27 1.27)
+				)
+			)
+		)
+		(property "KLC_S4.1" ""
+			(at 31.75 40.132 0)
+			(hide yes)
+			(show_name no)
+			(do_not_autoplace no)
+			(effects
+				(font
+					(size 1.27 1.27)
+				)
+			)
+		)
+		(pin "1"
+		)
+		(pin "2"
+		)
+		(instances
+			(project "PhaserPedalBoard"
+				(path "/121c4899-4e95-4dc0-b332-63e8ed3089d8/90bb61a7-a0ad-417b-bedc-65bd7068296f"
+					(reference "C25")
+					(unit 1)
+				)

Commit message: details and datasheets
Parts:
- removed C16: 100n, Capacitor_SMD:C_0805_2012Metric, symbol Device:C
- removed C19: 100u, Capacitor_THT:CP_Radial_D5.0mm_P2.50mm, symbol Device:C_Polarized_US
- removed C25: 10u, Capacitor_SMD:C_0805_2012Metric, symbol Device:C
- removed C26: 470u, Capacitor_THT:CP_Radial_D6.3mm_P2.50mm, symbol Device:C_Polarized_US
- removed J2: IO, symbol Connector:Conn_01x08_Pin
- removed NT1: NetTie_2, NetTie:NetTie-2_SMD_Pad0.5mm, symbol Device:NetTie_2
- removed R40: 22, Resistor_SMD:R_0805_2012Metric, symbol Device:R_US
- added C1: 220u, symbol Device:C_Polarized_Small_US
- added C18: 100n, Capacitor_SMD:C_0805_2012Metric, symbol Device:C
- added J1: Footswitch, symbol Connector:Conn_01x06_Pin
- added J7: PowerJack, Connector_BarrelJack:BarrelJack_Horizontal, symbol Connector:Barrel_Jack_Switch
- added R147: 22, Resistor_SMD:R_0805_2012Metric, symbol Device:R_US
Connections:
- net -9V is gone; now on net GND: C123.2, C124.2, R145.1, U1.2 (GND)
- net +3.3V: now also R147.2
- net BYP_IN: now also J1.3 (Pin_3)
- net FX_IN: now also J1.1 (Pin_1)
- net FX_OUT: now also J1.2 (Pin_2)
- net GND: now also C1.2, C18.1, J1.4 (Pin_4), J1.6 (Pin_6), J7.1, J7.3
- net TAP_IN: now also J1.5 (Pin_5)
- net VCC: now also U4.3 (VI), C18.2, J7.2
- net +9V renamed +12V
- net +12V: no longer U4.3 (VI)
- new net +3.3VA: C1.1, R147.1
Other:
- moved on the sheet: C17, C24, U4

Commit message: DAC stage looks good in sim
Parts:
- removed J1: Footswitch, symbol Connector:Conn_01x06_Pin

Commit message: rough schematic
Other:
- note added: "Power Jack"
- note removed: "IO/Power Header"
Changed lines of the file:
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@@
 		)
 	)
-	(text "IO/Power Header"
+	(text "Power Jack"
 		(exclude_from_sim no)
-		(at 38.1 23.876 0)
+		(at 30.988 24.13 0)
 		(effects
 			(font

Commit message: rough layout
Parts:
- C1: footprint (none) -> Capacitor_THT:CP_Radial_D7.5mm_P2.50mm
Changed lines of the file:
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@@
 			)
 		)
-		(property "Footprint" ""
+		(property "Footprint" "Capacitor_THT:CP_Radial_D7.5mm_P2.50mm"
 			(at 191.262 50.8 0)
 			(hide yes)

Commit message: routing w DRC passing
Parts:
- C1: value 220u -> 100u; footprint Capacitor_THT:CP_Radial_D7.5mm_P2.50mm -> Capacitor_THT:CP_Radial_D6.3mm_P2.50mm
Changed lines of the file:
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@@
 			)
 		)
-		(property "Value" "220u"
+		(property "Value" "100u"
 			(at 194.31 51.6381 0)
 			(show_name no)
@@
 			)
 		)
-		(property "Footprint" "Capacitor_THT:CP_Radial_D7.5mm_P2.50mm"
+		(property "Footprint" "Capacitor_THT:CP_Radial_D6.3mm_P2.50mm"
 			(at 191.262 50.8 0)
 			(hide yes)
